File: electronic/vfo-do.kicad_sch (KiCad schematic)
At the start: 24 parts, among them P1 12V in, P2 DWN, P3 Si5351, P4 Encoder, P5 GPS, P6 UP, P7 Band, P8 DIS GPS, P8 Reset, U1 24AA02-OT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

Commit message: electronics changes for PCB
Parts:
- removed C7: 100n, Capacitors_SMD:C_1206_HandSoldering, symbol vfo-do-rescue:C
- removed P2: DWN, Connectors_Molex:Molex_KK-6410-02_02x2.54mm_Straight, symbol vfo-do-rescue:CONN_01X02
- removed P3: Si5351, Connectors_Molex:Molex_KK-6410-07_07x2.54mm_Straight, symbol vfo-do-rescue:CONN_01X07
- removed P4: Encoder, Connectors_Molex:Molex_KK-6410-04_04x2.54mm_Straight, symbol vfo-do-rescue:CONN_01X04
- removed P5: GPS, Connectors_Molex:Molex_KK-6410-04_04x2.54mm_Straight, symbol vfo-do-rescue:CONN_01X04
- removed P6: UP, Connectors_Molex:Molex_KK-6410-02_02x2.54mm_Straight, symbol vfo-do-rescue:CONN_01X02
- removed P7: Band, Connectors_Molex:Molex_KK-6410-02_02x2.54mm_Straight, symbol vfo-do-rescue:CONN_01X02
- removed P8: Reset, Connectors_Molex:Molex_KK-6410-02_02x2.54mm_Straight, symbol vfo-do-rescue:CONN_01X02
- removed P8: DIS GPS, Connectors_Molex:Molex_KK-6410-02_02x2.54mm_Straight, symbol vfo-do-rescue:CONN_01X02
- removed U1: 24AA02-OT, Package_TO_SOT_SMD:SOT-23-5, symbol Memory_EEPROM:24AA02-OT
- removed U4: Arduino_Nano, arduino:arduino_nano, symbol vfo-do-rescue:Arduino_Nano
- added A1: Arduino_Nano_Socket, PCM_arduino-library:Arduino_Nano_Socket, symbol PCM_arduino-library:Arduino_Nano_Socket
- added J1: Commands, Connector_Molex:Molex_KK-254_AE-6410-04A_1x04_P2.54mm_Vertical, symbol Connector_Generic:Conn_01x04
- added J2: Dis GPS + Reset, Connector_Molex:Molex_KK-254_AE-6410-03A_1x03_P2.54mm_Vertical, symbol Connector_Generic:Conn_01x03
- added J3: Screen, Connector_Molex:Molex_KK-254_AE-6410-04A_1x04_P2.54mm_Vertical, symbol Connector_Generic:Conn_01x04
- added J4: SI5351, Connector_Molex:Molex_KK-254_AE-6410-05A_1x05_P2.54mm_Vertical, symbol Connector_Generic:Conn_01x05
- added J5: Encodeur, Connector_Molex:Molex_KK-254_AE-6410-04A_1x04_P2.54mm_Vertical, symbol Connector_Generic:Conn_01x04
- added J6: GPS, Connector_Molex:Molex_KK-254_AE-6410-04A_1x04_P2.54mm_Vertical, symbol Connector_Generic:Conn_01x04
- C1, C2, C6: footprint Capacitors_SMD:C_1206_HandSoldering -> Capacitor_THT:C_Disc_D5.0mm_W2.5mm_P5.00mm
- C3: renamed from C9; footprint Capacitors_SMD:C_1206_HandSoldering -> Capacitor_THT:C_Disc_D5.0mm_W2.5mm_P5.00mm
- C4: renamed from C10; footprint Capacitors_SMD:C_1206_HandSoldering -> Capacitor_THT:C_Disc_D5.0mm_W2.5mm_P5.00mm
- C5: renamed from C3; footprint Capacitors_SMD:C_1206_HandSoldering -> Capacitor_THT:C_Disc_D5.0mm_W2.5mm_P5.00mm
- C7: renamed from C5; footprint Capacitors_SMD:C_1206_HandSoldering -> Capacitor_THT:C_Disc_D5.0mm_W2.5mm_P5.00mm
- D1: footprint Diodes_SMD:SMB_Handsoldering -> Diode_THT:D_DO-41_SOD81_P7.62mm_Horizontal
- P1: value 12V in -> PWR IN; footprint Connectors_Molex:Molex_KK-6410-02_02x2.54mm_Straight -> Connector_Molex:Molex_KK-254_AE-6410-02A_1x02_P2.54mm_Vertical
- renumbered U2 to U1, U6 to U2, U5 to U3, U3 to U4
Connections:
- net GND: now also A1.GND1 (GND), A1.GND2 (GND), J1.4 (Pin_4), J2.1 (Pin_1), J3.4 (Pin_4), J4.2 (Pin_2), J5.1 (Pin_1), J6.4 (Pin_4)
- net at C7.1: now also A1.5V
- net at C2.1, U1.3 (VO), U2.1 (VI)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: now also A1.VIN
- net at C6.1, U2.3 (VO): now also J6.1 (Pin_1)
- net at C3.1, U3.3 (VO): now also J3.1 (Pin_1); no longer C5.2
- net at C4.1, U4.3 (VO): now also C5.2, J4.1 (Pin_1)
- new net: A1.D2 (D2_INT0), J6.3 (Pin_3)
- new net: A1.D3 (D3_INT1), J5.2 (Pin_2)
- new net: A1.D4, J5.3 (Pin_3)
- new net: A1.D5, J5.4 (Pin_4)
- new net: A1.A0, J1.1 (Pin_1)
- new net: A1.A1, J1.2 (Pin_2)
- new net: A1.A3, J1.3 (Pin_3)
- new net: A1.D7, J2.2 (Pin_2)
- new net: A1.RST1 (RESET), J2.3 (Pin_3)
- new net CLK0: A1.D6, J4.5 (Pin_5)
- new net RX GPS: A1.D0 (D0/RX), J6.2 (Pin_2)
- new net SCL: A1.A5 (A5/SCL), J3.3 (Pin_3), J4.4 (Pin_4)
- new net SDA: A1.A4 (A4/SDA), J3.2 (Pin_2), J4.3 (Pin_3)
- no-connect marks 10 -> 0
Other:
- note added: "1 - Down 2 - UP 3 - Band 4 - GND"
- note added: "1 - GND 2 - Disable GPS 3 - Reset"
- note added: "D0/RX GPS RX (this pin may differ on the Nano board) D1 D2 GPS 1pps input D3 Rotary encoder pin A D4 Rotary encoder pin B D5 2.5 MHz input from Si5351 CLK0 pin D6 Frequency resolution button D7 Disable GPS D8 D9 D10 D11 D12 D13 A0/D14 Decrease frequency button A1/D15 Increase frequency button A2/D16 Offset enable A3/D17 Band Select button A4/D18 Si5351 SDA - I2C LCD SDA A5/D19 Si5351 SCL - I2C LC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"
- note removed: "+5"
- note removed: "8V"
- note removed: "LDO 5V"
- note removed: "LDO Osc."
- note removed: "Neo 6/7"
- moved on the sheet: C1, C2, C3, C4, C5, C6, C7, D1, P1, U1, U2, U3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
